Commit message: add some notes

File: src/mrobot_gazebo/urdf/mrobot_body.urdf.xacro (robot description, xacro)
@@ -1,4 +1,5 @@
 <?xml version="1.0"?>
-<robot name="mrobot" xmlns:xacro="http://www.ros.org/wiki/xacro">
+<robot name="mrobot"
+    xmlns:xacro="http://www.ros.org/wiki/xacro">
     <!-- Defining the colors used in this robot -->
     <material name="Black">
@@ -18,28 +19,26 @@
     <xacro:property name="M_PI" value="3.1415926535897931" />
     <!-- Main body length, width, height and mass -->
-    <xacro:property name="base_mass"        value="0.5" />
+    <xacro:property name="base_mass" value="0.5" />
     <xacro:property name="base_link_radius" value="0.13"/>
     <xacro:property name="base_link_length" value="0.005"/>
     <xacro:property name="motor_x" value="-0.05"/>
     <!-- Caster radius and mass -->
-    <xacro:property name="caster_radius"          value="0.016" />
-    <xacro:property name="caster_mass"            value="0.01" />
-    <xacro:property name="caster_joint_origin_x"  value="-0.12" />
+    <xacro:property name="caster_radius" value="0.016" />
+    <xacro:property name="caster_mass" value="0.01" />
+    <xacro:property name="caster_joint_origin_x" value="-0.12" />
     <!-- Wheel radius, height and mass -->
     <xacro:property name="wheel_radius" value="0.033" />
     <xacro:property name="wheel_height" value="0.017" />
-    <xacro:property name="wheel_mass"   value="0.1" />
+    <xacro:property name="wheel_mass" value="0.1" />
     <!-- plate height and mass -->
-    <xacro:property name="plate_mass"   value="0.05"/>
+    <xacro:property name="plate_mass" value="0.05"/>
     <xacro:property name="plate_height" value="0.07"/>
-    <xacro:property name="standoff_x"   value="0.12"/>
-    <xacro:property name="standoff_y"   value="0.10"/>
+    <xacro:property name="standoff_x" value="0.12"/>
+    <xacro:property name="standoff_y" value="0.10"/>
     <!-- Macro for inertia matrix -->
     <xacro:macro name="sphere_inertial_matrix" params="m r">
         <inertial>
             <mass value="${m}" />
-            <inertia ixx="${2*m*r*r/5}" ixy="0" ixz="0"
-                iyy="${2*m*r*r/5}" iyz="0"
-                izz="${2*m*r*r/5}" />
+            <inertia ixx="${2*m*r*r/5}" ixy="0" ixz="0" iyy="${2*m*r*r/5}" iyz="0" izz="${2*m*r*r/5}" />
         </inertial>
     </xacro:macro>
@@ -47,7 +46,5 @@
         <inertial>
             <mass value="${m}" />
-            <inertia ixx="${m*(3*r*r+h*h)/12}" ixy = "0" ixz = "0"
-                iyy="${m*(3*r*r+h*h)/12}" iyz = "0"
-                izz="${m*r*r/2}" />
+            <inertia ixx="${m*(3*r*r+h*h)/12}" ixy = "0" ixz = "0" iyy="${m*(3*r*r+h*h)/12}" iyz = "0" izz="${m*r*r/2}" />
         </inertial>
     </xacro:macro>
@@ -55,7 +52,5 @@
         <inertial>
             <mass value="${m}" />
-            <inertia ixx="${m*(h*h+d*d)/12}" ixy = "0" ixz = "0"
-                iyy="${m*(w*w+d*d)/12}" iyz = "0"
-                izz="${m*(w*w+h*h)/12}" />
+            <inertia ixx="${m*(h*h+d*d)/12}" ixy = "0" ixz = "0" iyy="${m*(w*w+d*d)/12}" iyz = "0" izz="${m*(w*w+h*h)/12}" />
         </inertial>
     </xacro:macro>
@@ -77,5 +72,5 @@
                 </geometry>
             </collision>
-            <cylinder_inertial_matrix  m="${wheel_mass}" r="${wheel_radius}" h="${wheel_height}" />
+            <cylinder_inertial_matrix m="${wheel_mass}" r="${wheel_radius}" h="${wheel_height}" />
         </link>
         <gazebo reference="wheel_${lr}_link">
@@ -115,5 +110,5 @@
                 <origin xyz="0 0 0 " rpy="0 0 0" />
             </collision>
-            <sphere_inertial_matrix  m="${caster_mass}" r="${caster_radius}" />
+            <sphere_inertial_matrix m="${caster_mass}" r="${caster_radius}" />
         </link>
         <gazebo reference="${fb}_caster_link">
@@ -129,5 +124,5 @@
     <xacro:macro name="plate" params="num parent">
         <link name="plate_${num}_link">
-            <cylinder_inertial_matrix  m="0.1" r="${base_link_radius}" h="${base_link_length}" />
+            <cylinder_inertial_matrix m="0.1" r="${base_link_radius}" h="${base_link_length}" />
             <visual>
                 <origin xyz=" 0 0 0 " rpy="0 0 0" />
@@ -164,7 +159,5 @@
                 <mass value="0.001" />
                 <origin xyz="0 0 0" />
-                <inertia ixx="0.0001" ixy="0.0" ixz="0.0"
-          iyy="0.0001" iyz="0.0"
-          izz="0.0001" />
+                <inertia ixx="0.0001" ixy="0.0" ixz="0.0" iyy="0.0001" iyz="0.0" izz="0.0001" />
             </inertial>
             <visual>
@@ -204,5 +197,5 @@
         <!--Actual body/chassis of the robot-->
         <link name="base_link">
-            <cylinder_inertial_matrix  m="${base_mass}" r="${base_link_radius}" h="${base_link_length}" />
+            <cylinder_inertial_matrix m="${base_mass}" r="${base_link_radius}" h="${base_link_length}" />
             <visual>
                 <origin xyz=" 0 0 0" rpy="0 0 0" />
@@ -223,8 +216,8 @@
         </gazebo>
         <!-- Wheel Definitions -->
-        <wheel lr="right"  translateY="1" />
-        <wheel lr="left"  translateY="-1" />
+        <wheel lr="right" translateY="1" />
+        <wheel lr="left" translateY="-1" />
         <!-- Casters Definitions -->
-        <caster fb="front"  translateX="-1" />
+        <caster fb="front" translateX="-1" />
         <!-- plates and standoff Definitions -->
         <mrobot_standoff_2in parent="base_link" number="1" x_loc="-${standoff_x/2 + 0.03}" y_loc="-${standoff_y - 0.03}" z_loc="${plate_height/2}"/>
@@ -237,6 +230,6 @@
         <mrobot_standoff_2in parent="standoff_2in_4_link" number="8" x_loc="0" y_loc="0" z_loc="${plate_height}"/>
         <!-- plate Definitions -->
-        <plate num="1"  parent="base_link" />
-        <plate num="2"  parent="plate_1_link" />
+        <plate num="1" parent="base_link" />
+        <plate num="2" parent="plate_1_link" />
         <!-- controller -->
         <gazebo>
